File: dandelion_circuit/dandelion_circuit.sch (KiCad schematic (older format))
At the start: 49 parts

Commit message: removed undervoltage protection and added power mux ic to handle solar and USB input
Parts:
- added C?: 22u, symbol Device:C
- added C?: 100n, symbol Device:C
- added C?: 47u, symbol Device:C
- added L?: 4.7u, symbol Device:L
- added R?: 10k, symbol Device:R
- added R?: 56.2k, symbol Device:R
- added U?: TPS561201, Package_TO_SOT_SMD:SOT-23-6, symbol Regulator_Switching:TPS561201
- U? (x5): symbol smallIrrigationCircuit-rescue:MAX14626-Power_Protection -> dandelion_circuit-rescue:MAX14626-Power_Protection-smallIrrigationCircuit-rescue
Connections:
- net labels added: 5V
- wire segments 282 -> 305
