File: dandelion_circuit/dandelion_circuit.kicad_sch (KiCad schematic)
At the start: 112 parts, among them J1 MOLEX 733910083, J2 USB_B_Micro, J3 Micro_SD_Card, J4 Screw_Terminal_01x10, J5 S_NODE_SOLAR_INPUT, J6 Conn_01x02, Q1 SSM3J332R, SW1 Reset, SW2 BTN 1, SW3 SW_DIP_x03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

Commit message: Final circuit design
Parts:
- removed C16: 100n, Capacitor_SMD:C_0402_1005Metric, symbol Device:C
- removed C18, C21: 4.7u, Capacitor_SMD:C_0805_2012Metric, symbol Device:C
- removed J3: Micro_SD_Card, symbol Connector:Micro_SD_Card
- removed J5: S_NODE_SOLAR_INPUT, symbol Connector:Screw_Terminal_01x02
- removed JP1: EN, Jumper:SolderJumper-3_P1.3mm_Open_Pad1.0x1.5mm, symbol Device:Jumper_NC_Dual
- removed JP2: SETI, Jumper:SolderJumper-2_P1.3mm_Open_Pad1.0x1.5mm, symbol Device:Jumper
- removed R14, R19: 2.2M, symbol Device:R
- removed R15: 169k, symbol Device:R
- removed R16: 100k, symbol Device:R
- removed R20: 536k, symbol Device:R
- removed R21: 5.76k, symbol Device:R
- removed RN1: 10k, symbol Device:R_Pack05
- removed RN2: 100, symbol Device:R_Pack05
- removed U7: MAX14626, Package_DFN_QFN:DFN-6-1EP_3x3mm_P1mm_EP1.5x2.4mm, symbol dandelion_circuit-rescue:MAX14626-Power_Protection-smallIrrigationCircuit-rescue
- removed U9: MAX14573EUDT, SOP65P637X110-14N, symbol MAX14573EUDT:MAX14573EUDT
- added J3: Conn_01x02, Connector_PinHeader_2.00mm:PinHeader_1x02_P2.00mm_Vertical, symbol Connector_Generic:Conn_01x02
- added J5: Conn_01x04_Male, Connector_PinHeader_1.27mm:PinHeader_1x04_P1.27mm_Vertical, symbol Connector:Conn_01x04_Male
- added RN1: 10k, Resistor_SMD:R_Array_Convex_4x0603, symbol Device:R_Pack04
- added RN2: 160, Resistor_SMD:R_Array_Convex_4x0603, symbol Device:R_Pack04
- added TP1, TP10, TP11, TP12, TP13, TP2, TP3, TP4, TP5, TP6, TP7, TP8, TP9: TestPoint, TestPoint:TestPoint_Pad_2.0x2.0mm, symbol Connector:TestPoint
- C32: value 100n -> 22u
- J1: footprint Connector_Coaxial:SMA_Molex_73251-2200_Horizontal -> Connector_Coaxial:U.FL_Molex_MCRF_73412-0110_Vertical
- J2: footprint Connector_USB:USB_Micro-B_Molex_47346-0001 -> Connector_USB:USB_Micro-B_Molex-105133-0031
- J4: footprint (none) -> Connector_Phoenix_MSTB:Connector_Phoenix_MKKDSN
- J6: footprint (none) -> Connector_PinHeader_2.00mm:PinHeader_1x02_P2.00mm_Vertical
- L4: footprint (none) -> Inductor_SMD:Inductor_Sunlord_MWSA0603
- L5: footprint (none) -> Inductor_SMD:Sunlord_MWSA0503S
- R1, R17, R18, R2, R22, R23, R24, R25, R26, R27, R28, R3, R4, R5, R6, R7, R9: footprint (none) -> Resistor_SMD:R_0402_1005Metric
- R10: footprint (none) -> Resistor_SMD:R_0603_1608Metric
- R11: value 1.82k -> 1.54k; footprint (none) -> Resistor_SMD:R_0603_1608Metric
- R12: value 1.47k -> 1.18k; footprint (none) -> Resistor_SMD:R_0603_1608Metric
- R13, R8: value 1k -> 10k; footprint (none) -> Resistor_SMD:R_0402_1005Metric
- R14, R15, R16, R19, R20: renamed from R?; footprint (none) -> Resistor_SMD:R_0402_1005Metric
- SW1, SW2: footprint (none) -> Button_Switch_SMD:SW_Push_1P1T_NO_Vertical_Wuerth_434133025816
- SW3: footprint (none) -> Button_Switch_SMD:SW_DIP_SPSTx03_Slide_KingTek_DSHP03TJ_W5.25mm_P1.27mm_JPin
- SW4: footprint (none) -> Button_Switch_SMD:SW_SPDT_PCM12
- U13: footprint SON-6 -> TPD4E004DRYR:SON-6
- U8: footprint (none) -> Package_DFN_QFN:VQFN-16-1EP_3x3mm_P0.5mm_EP1.68x1.68mm_ThermalVias
- U9: renamed from U?; footprint IC_TPS2121RUXR -> TPS2121RUXR:IC_TPS2121RUXR
- Y1: footprint (none) -> Crystal:Crystal_SMD_Abracon_ABM10-4Pin_2.5x2.0mm
- gave numbers to parts that had none: 4
Connections:
- net +3V3: now also J5.4 (Pin_4), TP11.1
- net ADC_0: now also RN1.1 (R1.1)
- net ADC_0_IN: now also RN1.8 (R1.2), RN2.1 (R1.1), TP6.1
- net ADC_1: now also RN1.2 (R2.1)
- net ADC_1_IN: now also RN1.7 (R2.2), RN2.2 (R2.1), TP5.1
- net ADC_2: now also RN1.3 (R3.1)
- net ADC_2_IN: now also RN1.6 (R3.2), RN2.3 (R3.1), TP4.1
- net ADC_3: now also RN1.4 (R4.1)
- net ADC_3_IN: now also RN1.5 (R4.2), RN2.4 (R4.1), TP3.1
- net GND: now also U12.5 (SYNC), U8.17 (PAD), U8.8 (VSS), J3.2 (Pin_2), J5.1 (Pin_1), RN2.5 (R4.2), RN2.6 (R3.2), RN2.7 (R2.2), RN2.8 (R1.2); no longer J4.2 (Pin_2), J4.4 (Pin_4), J4.6 (Pin_6), J4.8 (Pin_8)
- net ID_BIT_0: now also U2.27 (PB6); no longer U2.28 (PB7)
- net ID_BIT_1: now also U2.26 (PB5); no longer U2.27 (PB6)
- net ID_BIT_2: now also U2.25 (PB4); no longer U2.26 (PB5)
- net S_NODE_5V_SOLAR: now also TP10.1
- net S_NODE_CE: now also U2.15 (PB1); no longer U2.22 (PA14)
- net S_NODE_COMBINED_POWER: now also TP9.1
- net S_NODE_IRQ: now also U2.14 (PB0); no longer U2.21 (PA13)
- net S_NODE_P_MUX_OUT: now also TP12.1
- net S_NODE_SS: now also U2.28 (PB7)
- net S_NODE_USB_POWER: now also TP2.1
- net S_NODE_VBAT: now also J3.1 (Pin_1)
- net at U2.18 (VDDIO2): now also TP1.1
- net S_NODE_SOLAR_INPUT: now reaches J4.9 (Pin_9)
- net S_NODE_SOLAR_INPUT: now also Q1.3 (D), TP7.1
- net 12V renamed S_NODE_12V
- net S_NODE_12V: now also J4.2 (Pin_2), J4.4 (Pin_4), J4.6 (Pin_6), J4.8 (Pin_8), TP13.1
- net ADC_4: no longer names the net of U2.10 (PA4)
- net OUVP_VIN_1 renamed S_NODE_SOLAR_OUTPUT
- net S_NODE_SOLAR_OUTPUT: now also TP8.1
- new net S_NODE_SWCLK: J5.2 (Pin_2), U2.22 (PA14)
- new net S_NODE_SWDIO: J5.3 (Pin_3), U2.21 (PA13)
- no-connect marks 6 -> 3
Other:
- note added: "Decoupljng capacitors needed?"
- note added: "remember to add the serial wire debug interface"
- note removed: "Over Voltage Under Voltage protection circuit (6-17V) output"
